Commit message: Updated the files

File: bot_description/urdf/bot.urdf.xacro (robot description, xacro)
@@ -403,10 +403,53 @@
   <gazebo reference="imu_link">
     <sensor name="imu" type="imu">
-      <always_on>1</always_on>
-      <update_rate>50</update_rate>
+      <always_on>true</always_on>
+      <update_rate>100</update_rate>  <!-- Higher rate for better fusion -->
       <visualize>true</visualize>
-      <topic>imu</topic>
+      <topic>/imu</topic>         <!-- Standard IMU topic -->
       <enable_metrics>true</enable_metrics>
       <gz_frame_id>imu_link</gz_frame_id>
+      <!-- Enhanced IMU parameters for accurate sensing -->
+      <imu>
+        <angular_velocity>
+          <x>
+            <noise type="gaussian">
+              <mean>0.0</mean>
+              <stddev>2e-4</stddev>
+            </noise>
+          </x>
+          <y>
+            <noise type="gaussian">
+              <mean>0.0</mean>
+              <stddev>2e-4</stddev>
+            </noise>
+          </y>
+          <z>
+            <noise type="gaussian">
+              <mean>0.0</mean>
+              <stddev>2e-4</stddev>
+            </noise>
+          </z>
+        </angular_velocity>
+        <linear_acceleration>
+          <x>
+            <noise type="gaussian">
+              <mean>0.0</mean>
+              <stddev>1.7e-2</stddev>
+            </noise>
+          </x>
+          <y>
+            <noise type="gaussian">
+              <mean>0.0</mean>
+              <stddev>1.7e-2</stddev>
+            </noise>
+          </y>
+          <z>
+            <noise type="gaussian">
+              <mean>0.0</mean>
+              <stddev>1.7e-2</stddev>
+            </noise>
+          </z>
+        </linear_acceleration>
+      </imu>
     </sensor>
   </gazebo>
@@ -419,40 +462,46 @@
     </sensor>
   </gazebo>
- <!-- Gazebo wheel physics -->
+ <!-- Optimized Gazebo wheel physics for accurate odometry -->
+  <!-- Front wheels Free-rolling, lower friction for Ackermann steering -->
   <gazebo reference="base_front_left_wheel">
-    <mu1>1.2</mu1>
-    <mu2>1.0</mu2>
-    <kp>20000.0</kp>
-    <kd>20.0</kd>
-    <minDepth>0.001</minDepth>
-    <maxVel>100</maxVel>
+    <mu1>0.8</mu1>        <!-- Lower friction for free-rolling front wheels -->
+    <mu2>0.6</mu2>        <!-- Reduced lateral friction -->
+    <kp>50000.0</kp>      <!-- Higher contact stiffness for less slip -->
+    <kd>50.0</kd>         <!-- Higher damping for stability -->
+    <minDepth>0.0005</minDepth>  <!-- Smaller penetration depth -->
+    <maxVel>10.0</maxVel>        <!-- Lower max velocity for stability -->
+    <fdir1>0 -1 0</fdir1>        <!-- Primary friction direction -->
+    <material>Gazebo/Grey</material>
+  </gazebo>
+  <gazebo reference="base_front_right_wheel">
+    <mu1>0.8</mu1>
+    <mu2>0.6</mu2>
+    <kp>50000.0</kp>
+    <kd>50.0</kd>
+    <minDepth>0.0005</minDepth>
+    <maxVel>10.0</maxVel>
     <fdir1>0 -1 0</fdir1>
-  </gazebo>
-  <gazebo reference="base_front_right_wheel">
-    <mu1>1.2</mu1>
-    <mu2>1.0</mu2>
-    <kp>20000.0</kp>
-    <kd>20.0</kd>
-    <minDepth>0.001</minDepth>
-    <maxVel>100</maxVel>
+    <material>Gazebo/Grey</material>
+  </gazebo>
+  <!-- Rear wheels Drive wheels, optimized for no-slip control -->
+  <gazebo reference="base_back_left_wheel">
+    <mu1>1.8</mu1>        <!-- Higher friction for drive wheels -->
+    <mu2>1.5</mu2>        <!-- High lateral friction to prevent sliding -->
+    <kp>100000.0</kp>     <!-- Very high stiffness for accurate control -->
+    <kd>100.0</kd>        <!-- Higher damping for precise motion -->
+    <minDepth>0.0005</minDepth>  <!-- Smaller penetration depth -->
+    <maxVel>10.0</maxVel>        <!-- Lower max velocity for stability -->
+    <fdir1>0 -1 0</fdir1>        <!-- Primary friction direction -->
+    <material>Gazebo/Black</material>
+  </gazebo>
+  <gazebo reference="base_back_right_wheel">
+    <mu1>1.8</mu1>
+    <mu2>1.5</mu2>
+    <kp>100000.0</kp>
+    <kd>100.0</kd>
+    <minDepth>0.0005</minDepth>
+    <maxVel>10.0</maxVel>
     <fdir1>0 -1 0</fdir1>
-  </gazebo>
-  <gazebo reference="base_back_left_wheel">
-    <mu1>1.2</mu1>
-    <mu2>1.0</mu2>
-    <kp>20000.0</kp>
-    <kd>20.0</kd>
-    <minDepth>0.001</minDepth>
-    <maxVel>100</maxVel>
-    <fdir1>0 -1 0</fdir1>
-  </gazebo>
-  <gazebo reference="base_back_right_wheel">
-    <mu1>1.2</mu1>
-    <mu2>1.0</mu2>
-    <kp>20000.0</kp>
-    <kd>20.0</kd>
-    <minDepth>0.001</minDepth>
-    <maxVel>100</maxVel>
-    <fdir1>0 -1 0</fdir1>
+    <material>Gazebo/Black</material>
   </gazebo>
   <gazebo>

File: bot_description/urdf/bot_ros2_control.xacro (robot description, xacro)
@@ -23,21 +23,12 @@
       <state_interface name="velocity"/>
     </joint>
-    <!-- Wheel Joints
     <joint name="base_front_left_wheel_joint">
-      <command_interface name="velocity">
-        <param name="min">-10</param>
-        <param name="max">10</param>
-      </command_interface>
       <state_interface name="position"/>
       <state_interface name="velocity"/>
     </joint>
     <joint name="base_front_right_wheel_joint">
-      <command_interface name="velocity">
-        <param name="min">-10</param>
-        <param name="max">10</param>
-      </command_interface>
       <state_interface name="position"/>
       <state_interface name="velocity"/>
-    </joint> -->
+    </joint>
     <joint name="base_back_left_wheel_joint">
       <command_interface name="velocity">

Commit message: Update bot.urdf.xacro

File: bot_description/urdf/bot.urdf.xacro (robot description, xacro)
@@ -111,6 +111,6 @@
         <cylinder radius="0.175" length="0.13"/>
       </geometry>
-      <material name="red">
-        <color rgba="0.8 0.2 0.2 1"/>
+      <material name="grey">
+        <color rgba="0.5 0.5 0.5 1"/>
       </material>
     </visual>
@@ -140,6 +140,6 @@
         <cylinder radius="0.175" length="0.13"/>
       </geometry>
-      <material name="red">
-        <color rgba="0.8 0.2 0.2 1"/>
+      <material name="grey">
+        <color rgba="0.5 0.5 0.5 1"/>
       </material>
     </visual>
@@ -169,6 +169,6 @@
         <cylinder radius="0.175" length="0.13"/>
       </geometry>
-      <material name="red">
-        <color rgba="0.8 0.2 0.2 1"/>
+      <material name="black">
+        <color rgba="0.1 0.1 0.1 1"/>
       </material>
     </visual>
@@ -198,6 +198,6 @@
         <cylinder radius="0.175" length="0.13"/>
       </geometry>
-      <material name="red">
-        <color rgba="0.8 0.2 0.2 1"/>
+      <material name="black">
+        <color rgba="0.1 0.1 0.1 1"/>
       </material>
     </visual>
@@ -254,5 +254,5 @@
       <origin xyz="0 0 0" rpy="0 0 1.57079632679" />
       <geometry>
-         <mesh filename="file:///home/aditya-pachauri/prototype_autonomous_bot_cir_ws/src/bot_description/meshes/3dCamera.DAE" scale="1 1 1"/>
+         <mesh filename="file://$(find bot_description)/meshes/3dCamera.DAE" scale="1 1 1"/>
       </geometry>
     </visual>
@@ -265,5 +265,5 @@
   </link>
   <joint name="camera_joint" type="fixed">
-    <origin xyz="0.085 0 0.002" rpy="0 0.0 0"/>
+    <origin xyz="0 0.685 0.15" rpy="0 0.0 1.57079632679"/>
     <parent link="base_link"/>
     <child link="rgb_camera"/>
@@ -313,9 +313,8 @@
     <visual>
       <geometry>
-        <mesh filename="file:///home/aditya-pachauri/prototype_autonomous_bot_cir_ws/src/bot_description/meshes/lidar_3d_v1.dae" scale="1 1 1"/>
+        <mesh filename="file://$(find bot_description)/meshes/lidar_3d_v1.dae" scale="1 1 1"/>
       </geometry>
     </visual>
     <collision>
-      <origin xyz="0 0 0.03585" rpy="0 0 0"/>
       <geometry>
         <cylinder radius="0.0516" length="0.0717" />
@@ -347,5 +346,5 @@
   </link>
     <joint name="lidar_base_joint" type="fixed">
-    <origin xyz="0 0 0.02" rpy="0 0.0 3.14"/>
+    <origin xyz="0 0 0.25" rpy="0 0.0 0.0"/>
     <parent link="base_link"/>
     <child link="lidar_base"/>
@@ -353,6 +352,6 @@
   </joint>
   <joint name="laser_joint" type="fixed">
-    <origin xyz="0 0 0.046" rpy="0 0.0 3.14"/>
-    <parent link="base_link"/>
+    <origin xyz="0 0 0.027" rpy="0 0.0 0.0"/>
+    <parent link="lidar_base"/>
     <child link="laser_link"/>
     <axis xyz="0.0 0.0 1.0"/>
@@ -507,5 +506,5 @@
   <gazebo>
     <plugin filename="gz_ros2_control-system" name="gz_ros2_control::GazeboSimROS2ControlPlugin">
-      <parameters>/home/aditya-pachauri/prototype_autonomous_bot_cir_ws/src/bot_controller/config/bot_controller.yaml</parameters>
+      <parameters>$(find bot_controller)/config/bot_controller.yaml</parameters>
     </plugin>
     <plugin filename="gz-sim-imu-system" name="gz::sim::systems::Imu">

Commit message: Change wheel joint axis direction to positive Z

File: bot_description/urdf/bot.urdf.xacro (robot description, xacro)
@@ -184,5 +184,5 @@
     <child link="base_back_left_wheel"/>
     <origin xyz="-0.335 -0.51 -0.2075" rpy="0 1.57079632679 0"/>
-    <axis xyz="0 0 -1"/>
+    <axis xyz="0 0 1"/>
   </joint>
     <!-- ========== BACK RIGHTWHEEL ========== -->
@@ -213,5 +213,5 @@
     <child link="base_back_right_wheel"/>
     <origin xyz="0.335 -0.51 -0.2075" rpy="0 1.57079632679 0"/>
-    <axis xyz="0 0 -1"/>
+    <axis xyz="0 0 1"/>
   </joint>
 <!-- ============================================ -->

Commit message: Add files via upload

File: bot_description/urdf/bot.urdf.xacro (robot description, xacro)
@@ -9,10 +9,10 @@
       <origin xyz="0 0 0" rpy="0 0 0"/>
       <mass value="5"/>
-      <inertia ixx="0.829" ixy="0" ixz="0" iyy="0.063" iyz="0" izz="0.827"/>
+      <inertia ixx="0.144" ixy="0" ixz="0" iyy="0.857" iyz="0" izz="0.840"/>
     </inertial>
     <collision name="base_collision">
       <origin xyz="0 0 0" rpy="0 0 0"/>
       <geometry>
-        <box size="0.37 1.37 0.415"/>
+        <box size="1.37 0.37 0.415"/>
       </geometry>
       <surface>
@@ -28,5 +28,5 @@
       <origin xyz="0 0 0" rpy="0 0 0"/>
       <geometry>
-        <box  size="0.37 1.37 0.415"/>
+        <box  size="1.37 0.37 0.415"/>
       </geometry>
       <material name="blue">
@@ -66,7 +66,7 @@
     <parent link="base_link"/>
     <child link="base_front_left_steering"/>
-    <origin xyz="-0.265 0.39 -0.2075" rpy="0 1.57079632679 0"/>
+    <origin xyz="0.39 -0.265 -0.2075" rpy="-1.57079632679 0 0"/>
     <limit lower="-0.2616" upper="0.2616" effort="100" velocity="1.0"/>
-    <axis xyz="-1 0 0"/>
+    <axis xyz="0 1 0"/>
   </joint>
   <link name="base_front_right_steering">
@@ -95,7 +95,7 @@
     <parent link="base_link"/>
     <child link="base_front_right_steering"/>
-    <origin xyz="0.265 0.39 -0.2075" rpy="0 1.57079632679 0"/>
+    <origin xyz="0.39 0.265 -0.2075" rpy="-1.57079632679 0 0"/>
     <limit lower="-0.2616" upper="0.2616" effort="100" velocity="1.0"/>
-    <axis xyz="-1 0 0"/>
+    <axis xyz="0 1 0"/>
   </joint>
   <!-- ========== FRONT LEFTWHEEL ========== -->
@@ -183,5 +183,5 @@
     <parent link="base_link"/>
     <child link="base_back_left_wheel"/>
-    <origin xyz="-0.335 -0.51 -0.2075" rpy="0 1.57079632679 0"/>
+    <origin xyz="-0.51 -0.335 -0.2075" rpy="-1.57079632679 0 0"/>
     <axis xyz="0 0 1"/>
   </joint>
@@ -212,5 +212,5 @@
     <parent link="base_link"/>
     <child link="base_back_right_wheel"/>
-    <origin xyz="0.335 -0.51 -0.2075" rpy="0 1.57079632679 0"/>
+    <origin xyz="-0.51 0.335 -0.2075" rpy="-1.57079632679 0 0"/>
     <axis xyz="0 0 1"/>
   </joint>
@@ -241,5 +241,5 @@
     <parent link="base_link"/>
     <child link="bot_storage_base"/>
-    <origin xyz="0 0 0.2325" rpy="0 0 0"/>
+    <origin xyz="0 0 0.2325" rpy="0 0 1.57079632679"/>
   </joint>
 <!-- ============================================ -->
@@ -265,5 +265,5 @@
   </link>
   <joint name="camera_joint" type="fixed">
-    <origin xyz="0 0.685 0.15" rpy="0 0.0 1.57079632679"/>
+    <origin xyz="0.685 0 0.15" rpy="0 0 0"/>
     <parent link="base_link"/>
     <child link="rgb_camera"/>
